File: design_blocks/ckl-blocks.kicad_block/Chip Antenna 2.45GHz.kicad_block/Chip Antenna 2.45GHz.kicad_pcb (KiCad board)
At the start: 4 copper layers, 2 parts

Commit message: A few extra antennas
Parts:
- AE2: footprint nrf52:Walsin_RFANT3216120A5T -> PCM_ckl-misc:Walsin_RFANT3216120A5T
Changed lines of the file:
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@@
 		)
 	)
-	(footprint "nrf52:Walsin_RFANT3216120A5T"
+	(footprint "PCM_ckl-misc:Walsin_RFANT3216120A5T"
 		(layer "F.Cu")
 		(at 143.98 156.41 -90)
