File: libmanagement/libmanagement.kicad_sch (KiCad schematic)
At the start: 0 parts

Commit message: A few extra antennas
Parts:
- added AE1: Antenna_Chip, PCM_ckl-misc:Walsin_RFANT3216120A5T, symbol Device:Antenna_Chip
- added L1: 6.8nH, Inductor_SMD:L_0402_1005Metric, symbol Device:L
Connections:
- new net RF3: AE1.1 (FEED), L1.1
- no-connect marks 0 -> 1
Changed lines of the file:
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@@
 	(generator_version "10.0")
 	(paper "A4")
+	(no_connect
+		(at 120.65 63.5)
+	)
+	(wire
+		(pts
+			(xy 125.73 63.5) (xy 125.73 64.77)
+		)
+		(stroke
+			(width 0)
+			(type default)
+		)
+	)
+	(wire
+		(pts
+			(xy 125.73 64.77) (xy 130.81 64.77)
+		)
+		(stroke
+			(width 0)
+			(type default)
+		)
+	)
+	(label "RF3"
+		(at 125.73 64.77 0)
+		(effects
+			(font
+				(size 1.27 1.27)
+			)
+			(justify left bottom)
+		)
+	)
+	(symbol
+		(lib_id "Device:Antenna_Chip")
+		(at 123.19 60.96 0)
+		(mirror y)
+		(unit 1)
+		(body_style 1)
+		(exclude_from_sim no)
+		(in_bom yes)
+		(on_board yes)
+		(in_pos_files yes)
+		(dnp no)
+		(property "Reference" "AE1"
+			(at 118.11 57.1499 0)
+			(show_name no)
+			(do_not_autoplace no)
+			(effects
+				(font
+					(size 1.27 1.27)
+				)
+				(justify left)
+			)
+		)
+		(property "Value" "Antenna_Chip"
+			(at 118.11 59.6899 0)
+			(show_name no)
+			(do_not_autoplace no)
+			(effects
+				(font
+					(size 1.27 1.27)
+				)
+				(justify left)
+			)
+		)
+		(property "Footprint" "PCM_ckl-misc:Walsin_RFANT3216120A5T"
+			(at 125.73 56.515 0)
+			(hide yes)
+			(show_name no)
+			(do_not_autoplace no)
+			(effects
+				(font
+					(size 1.27 1.27)
+				)
+			)
+		)
+		(property "Datasheet" "C127629"
+			(at 125.73 56.515 0)
+			(hide yes)
+			(show_name no)
+			(do_not_autoplace no)
+			(effects
+				(font
+					(size 1.27 1.27)
+				)
+			)
+		)
+		(property "Description" "Ceramic chip antenna with pin for PCB trace"
+			(at 123.19 60.96 0)
+			(hide yes)
+			(show_name no)
+			(do_not_autoplace no)
+			(effects
+				(font
+					(size 1.27 1.27)
+				)
+			)
+		)
+		(property "LCSC Part #" "C127629"
+			(at 123.19 60.96 0)
+			(hide yes)
+			(show_name no)
+			(do_not_autoplace no)
+			(effects
+				(font
+					(size 1.27 1.27)
+				)
+			)
+		)
+		(pin "1"
+		)
+		(pin "2"
+		)
+		(instances
+			(project "libmanagement"
+				(path "/3167b783-bede-465f-b0cf-2ffbbf5b7fd6"
+					(reference "AE1")
+					(unit 1)
+				)
+			)
+			(project "nrf52"
+				(path "/7c3fbfcb-953e-4e2a-9a2f-c270f824b4f7"
+					(reference "AE2")
+					(unit 1)
+				)
+			)
+		)
+	)
+	(symbol
+		(lib_id "Device:L")
+		(at 134.62 64.77 90)
+		(unit 1)
+		(body_style 1)
+		(exclude_from_sim no)
+		(in_bom yes)
+		(on_board yes)
+		(in_pos_files yes)
+		(dnp no)
+		(property "Reference" "L1"
+			(at 134.62 59.69 90)
+			(show_name no)
+			(do_not_autoplace no)
+			(effects
+				(font
+					(size 1.27 1.27)
+				)
+			)
+		)
+		(property "Value" "6.8nH"
+			(at 134.62 62.23 90)
+			(show_name no)
+			(do_not_autoplace no)
+			(effects
+				(font
+					(size 1.27 1.27)
+				)
+			)
+		)
+		(property "Footprint" "Inductor_SMD:L_0402_1005Metric"
+			(at 134.62 64.77 0)
+			(hide yes)
+			(show_name no)
+			(do_not_autoplace no)
+			(effects
+				(font
+					(size 1.27 1.27)
+				)
+			)
+		)
+		(property "Datasheet" ""
+			(at 134.62 64.77 0)
+			(hide yes)
+			(show_name no)
+			(do_not_autoplace no)
+			(effects
+				(font
+					(size 1.27 1.27)
+				)
+			)
+		)
+		(property "Description" "Inductor"
+			(at 134.62 64.77 0)
+			(hide yes)
+			(show_name no)
+			(do_not_autoplace no)
+			(effects
+				(font
+					(size 1.27 1.27)
+				)
+			)
+		)
+		(property "LCSC Part #" "C96056"
+			(at 134.62 64.77 90)
+			(hide yes)
+			(show_name no)
+			(do_not_autoplace no)
+			(effects
+				(font
+					(size 1.27 1.27)
+				)
+			)
+		)
+		(pin "1"
+		)
+		(pin "2"
+		)
+		(instances
+			(project "libmanagement"
+				(path "/3167b783-bede-465f-b0cf-2ffbbf5b7fd6"
+					(reference "L1")
+					(unit 1)
+				)
+			)
+			(project "nrf52"
+				(path "/7c3fbfcb-953e-4e2a-9a2f-c270f824b4f7"
+					(reference "L5")
+					(unit 1)
+				)
+			)
+		)
+	)
+	(group "Chip Antenna 2.45GHz"
+		(lib_id "WIP_ckl-blocks:Chip Antenna 2.45GHz")
+		(members "1920ba6c-2649-49ee-92bf-ae2def7b3dc3" "376ab7f6-4de2-417c-bc49-5829df0f47f7"
+			"654e6cd0-df59-46e5-b19a-970a90776c4f" "9628e3b6-bd5d-4811-b0eb-cd6d47ef7beb"
+			"9c3083bf-82df-4274-86a9-5760a7baea61" "e91dd93e-a42b-45f4-8486-fa4a81d9d13d"
+		)
+	)
 	(sheet_instances
 		(path "/"
